File: Hardware/KiCad/CrowdAware Node Rev1.1.kicad_pcb (KiCad board)
At the start: 2 copper layers, 80 x 40 mm, 10 parts, among them J1 2 pcs 1x18 socket 2.54mm

Commit message: Finalize verified CrowdAware Node Rev 1.1 hardware
Parts:
- A1: footprint Library:MLX90640ESF-BAA-000-TU -> IoT_Thermal:MLX90640ESF-BAA-000-TU
- C1, C2: footprint Capacitor_SMD:C_1206_3216Metric_Pad1.33x1.80mm_HandSolder -> IoT_Thermal:C_1206_3216Metric_Pad1.33x1.80mm_HandSolder
- H1, H2, H3, H4: renamed from REF**; footprint MyLib:MountingHole_3.2mm_M3 -> MountingHole:MountingHole_3.2mm_M3
- J1: footprint Library:Connector_HeltecWiFiLoRa32v3 -> IoT_Thermal:Connector_HeltecWiFiLoRa32v3
- R1, R2: value 1k 0603 10% -> 1k 0603 5%; footprint MyLib:R_0603_1608Metric_Pad0.98x0.95mm_HandSolder -> IoT_Thermal:R_0603_1608Metric_Pad0.98x0.95mm_HandSolder
- moved C1 2.55 mm to (140.5, 78.5), turned to 0 degrees
- moved C2 2.50 mm to (140.5, 82.0), turned to 0 degrees
Connections:
- J1 pad 21: /SCL -> /SDA
- J1 pad 23: /SDA -> /SCL
Routing:
- net /SCL: track 56.9 -> 59.4 mm, vias 0 -> 1
- net /SDA: track 51.6 -> 53.0 mm, vias 0 -> 1
- removed copper zone on F.Cu, net V_EXT
