File: Hardware/KiCad/CrowdAware Node Rev1.1.kicad_sch (KiCad schematic)
At the start: 6 parts, among them J1 2 pcs 1x18 socket 2.54mm

Commit message: Finalize verified CrowdAware Node Rev 1.1 hardware
Parts:
- A1: footprint Library:MLX90640ESF-BAA-000-TU -> IoT_Thermal:MLX90640ESF-BAA-000-TU; symbol MLX90640ESF-BAA-000-TU:MLX90640ESF-BAA-000-TU -> IoT_Thermal:MLX90640ESF-BAA-000-TU
- C1, C2: footprint Capacitor_SMD:C_1206_3216Metric_Pad1.33x1.80mm_HandSolder -> IoT_Thermal:C_1206_3216Metric_Pad1.33x1.80mm_HandSolder; symbol MySymbols:C -> Device:C
- J1: footprint Library:Connector_HeltecWiFiLoRa32v3 -> IoT_Thermal:Connector_HeltecWiFiLoRa32v3; symbol MySymbols:Conn_02x18_Odd_Even -> IoT_Thermal:Heltec_WiFi_LoRa_32_V3_Headers
- R1, R2: value 1k 0603 10% -> 1k 0603 5%; footprint MyLib:R_0603_1608Metric_Pad0.98x0.95mm_HandSolder -> IoT_Thermal:R_0603_1608Metric_Pad0.98x0.95mm_HandSolder; symbol MySymbols:R -> Device:R
Connections:
- net SCL: now also J1.23 (Pin_23); no longer J1.21 (Pin_21)
- net SDA: now also J1.21 (Pin_21); no longer J1.23 (Pin_23)
Other:
- note added: "This board relies on the Heltec WiFi LoRa 32(V3) development board, which provides: - A built-in battery interface and USB charging circuit - On-board LoRa and WiFi support - A GPIO-controlled +3V3 source V_EXT (active low: drive GPIO36 low to enable) - Integrated RF and low-power circuitry"
- note removed: "This board for the most part relies on the Heltec WiFi LoRa 32(V3) development board, which in itself contains: - A built-in battery interface and BMS with USB charging - On-board LoRa and WiFi support - A GPIO-controlled +3V3 source V_EXT (High by default, disabled by driving GPIO36 low) - Good RF and low-power circuitry"
Changed lines of the file:
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@@
 	(title_block
 		(title "CrowdAware Node Rev1.1")
-		(date "2026-09-15")
+		(date "2026-09-16")
 		(rev "1.1")
 		(company "InnoWing IoT Team")
-		(comment 1 "Based on v1.0 by Ilo Japar; Rev1.1 thermal-layout update")
-	)
-	(text "This board for the most part relies on the Heltec WiFi LoRa 32(V3) development board,\nwhich in itself contains:\n- A built-in battery interface and BMS with USB charging\n- On-board LoRa and WiFi support\n- A GPIO-controlled +3V3 source V_EXT (High by default, disabled by driving GPIO36 low)\n- Good RF and low-power circuitry"
+		(comment 1 "Based on v1.0 by Ilo Japar; Rev1.1 thermal and routing update")
+	)
+	(text "This board relies on the Heltec WiFi LoRa 32(V3) development board, which provides:\n- A built-in battery interface and USB charging circuit\n- On-board LoRa and WiFi support\n- A GPIO-controlled +3V3 source V_EXT (active low: drive GPIO36 low to enable)\n- Integrated RF and low-power circuitry"
 		(exclude_from_sim no)
 		(at 19.05 24.13 0)
@@
 	(wire
 		(pts
-			(xy 134.62 66.04) (xy 154.94 66.04)
+			(xy 134.62 66.04) (xy 144.78 66.04)
+		)
+		(stroke
+			(width 0)
+			(type default)
+		)
+	)
+	(wire
+		(pts
+			(xy 152.4 66.04) (xy 154.94 66.04)
 		)
 		(stroke
@@
 	(wire
 		(pts
-			(xy 116.84 63.5) (xy 154.94 63.5)
+			(xy 116.84 63.5) (xy 144.78 63.5)
+		)
+		(stroke
+			(width 0)
+			(type default)
+		)
+	)
+	(wire
+		(pts
+			(xy 152.4 63.5) (xy 154.94 63.5)
 		)
 		(stroke
@@
 	)
 	(label "SDA"
-		(at 148.59 66.04 0)
+		(at 144.78 66.04 180)
 		(effects
 			(font
 				(size 1.27 1.27)
 			)
-			(justify left bottom)
+			(justify right bottom)
 		)
 	)
 	(label "SCL"
-		(at 148.59 63.5 0)
+		(at 144.78 63.5 180)
 		(effects
 			(font
 				(size 1.27 1.27)
 			)
+			(justify right bottom)
+		)
+	)
+	(label "SDA"
+		(at 152.4 63.5 0)
+		(effects
+			(font
+				(size 1.27 1.27)
+			)
 			(justify left bottom)
 		)
 	)
+	(label "SCL"
+		(at 152.4 66.04 0)
+		(effects
+			(font
+				(size 1.27 1.27)
+			)
+			(justify left bottom)
+		)
+	)
 	(symbol
-		(lib_id "MySymbols:Conn_02x18_Odd_Even")
+		(lib_id "IoT_Thermal:Heltec_WiFi_LoRa_32_V3_Headers")
 		(at 160.02 58.42 0)
 		(unit 1)
@@
 			)
 		)
-		(property "Footprint" "Library:Connector_HeltecWiFiLoRa32v3"
+		(property "Footprint" "IoT_Thermal:Connector_HeltecWiFiLoRa32v3"
 			(at 160.02 58.42 0)
 			(hide yes)
@@
 	)
 	(symbol
-		(lib_id "MySymbols:C")
+		(lib_id "Device:C")
 		(at 39.37 64.77 0)
 		(unit 1)
@@
 			)
 		)
-		(property "Footprint" "Capacitor_SMD:C_1206_3216Metric_Pad1.33x1.80mm_HandSolder"
+		(property "Footprint" "IoT_Thermal:C_1206_3216Metric_Pad1.33x1.80mm_HandSolder"
 			(at 40.3352 68.58 0)
 			(hide yes)
@@
 	)
 	(symbol
-		(lib_id "MySymbols:R")
+		(lib_id "Device:R")
 		(at 134.62 55.88 0)
 		(unit 1)
@@
 			)
 		)
-		(property "Value" "1k 0603 10%"
+		(property "Value" "1k 0603 5%"
 			(at 137.16 57.1499 0)
 			(show_name no)
@@
 			)
 		)
-		(property "Footprint" "MyLib:R_0603_1608Metric_Pad0.98x0.95mm_HandSolder"
+		(property "Footprint" "IoT_Thermal:R_0603_1608Metric_Pad0.98x0.95mm_HandSolder"
 			(at 132.842 55.88 90)
 			(hide yes)
@@
 	)
 	(symbol
-		(lib_id "MySymbols:R")
+		(lib_id "Device:R")
 		(at 116.84 55.88 0)
 		(unit 1)
@@
 			)
 		)
-		(property "Value" "1k 0603 10%"
+		(property "Value" "1k 0603 5%"
 			(at 119.38 57.1499 0)
 			(show_name no)
@@
 			)
 		)
-		(property "Footprint" "MyLib:R_0603_1608Metric_Pad0.98x0.95mm_HandSolder"
+		(property "Footprint" "IoT_Thermal:R_0603_1608Metric_Pad0.98x0.95mm_HandSolder"
 			(at 115.062 55.88 90)
 			(hide yes)
@@
 	)
 	(symbol
-		(lib_id "MLX90640ESF-BAA-000-TU:MLX90640ESF-BAA-000-TU")
+		(lib_id "IoT_Thermal:MLX90640ESF-BAA-000-TU")
 		(at 96.52 63.5 0)
 		(mirror y)
@@
 			)
 		)
-		(property "Footprint" "Library:MLX90640ESF-BAA-000-TU"
+		(property "Footprint" "IoT_Thermal:MLX90640ESF-BAA-000-TU"
 			(at 96.52 63.5 0)
 			(hide yes)
@@
 	)
 	(symbol
-		(lib_id "MySymbols:C")
+		(lib_id "Device:C")
 		(at 62.23 64.77 0)
 		(unit 1)
@@
 			)
 		)
-		(property "Footprint" "Capacitor_SMD:C_1206_3216Metric_Pad1.33x1.80mm_HandSolder"
+		(property "Footprint" "IoT_Thermal:C_1206_3216Metric_Pad1.33x1.80mm_HandSolder"
 			(at 63.1952 68.58 0)
 			(hide yes)
