File: Hardware/KiCad/HKU Thermal Node Rev1.1.kicad_pcb (KiCad board)
At the start: 2 copper layers, 80 x 40 mm, 10 parts, among them J1 2 pcs 1x18 socket 2.54mm

Commit message: Fix Rev 1.1 production blockers and rename hardware
Connections:
- J1 pad 21: /SDA -> unconnected-(J1-Pin_21-Pad21)
- J1 pad 23: /SCL -> unconnected-(J1-Pin_23-Pad23)
- J1 pad 5: unconnected-(J1-Pin_5-Pad5) -> /SCL
- J1 pad 7: unconnected-(J1-Pin_7-Pad7) -> /SDA
Routing:
- net /SCL: track 59.4 -> 81.5 mm, vias 1 -> 2
- net /SDA: track 53.0 -> 68.8 mm
Other:
- board text added: "HKU IoT Beyond Lab"
- board text added: "HKU Thermal Node"
- board text removed: "CrowdAware Node"
- board text removed: "HKU InnoWing IoT Team"
Changed lines of the file:
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@@
 	(paper "A5")
 	(title_block
-		(title "CrowdAware Node Rev1.1")
+		(title "HKU Thermal Node Rev1.1")
 		(date "2026-09-16")
 		(rev "1.1")
@@
 		(property ki_fp_filters "C_*")
 		(sheetname "/")
-		(sheetfile "CrowdAware Node Rev1.1.kicad_sch")
+		(sheetfile "HKU Thermal Node Rev1.1.kicad_sch")
 		(units
 			(unit
@@
 		)
 		(sheetname "/")
-		(sheetfile "CrowdAware Node Rev1.1.kicad_sch")
+		(sheetfile "HKU Thermal Node Rev1.1.kicad_sch")
 		(units
 			(unit
@@
 		(property ki_fp_filters "R_*")
 		(sheetname "/")
-		(sheetfile "CrowdAware Node Rev1.1.kicad_sch")
+		(sheetfile "HKU Thermal Node Rev1.1.kicad_sch")
 		(units
 			(unit
@@
 		(property ki_fp_filters "C_*")
 		(sheetname "/")
-		(sheetfile "CrowdAware Node Rev1.1.kicad_sch")
+		(sheetfile "HKU Thermal Node Rev1.1.kicad_sch")
 		(units
 			(unit
@@
 		(property ki_fp_filters "R_*")
 		(sheetname "/")
-		(sheetfile "CrowdAware Node Rev1.1.kicad_sch")
+		(sheetfile "HKU Thermal Node Rev1.1.kicad_sch")
 		(units
 			(unit
@@
 		(property ki_fp_filters "Connector*:*_2x??_*")
 		(sheetname "/")
-		(sheetfile "CrowdAware Node Rev1.1.kicad_sch")
+		(sheetfile "HKU Thermal Node Rev1.1.kicad_sch")
 		(units
 			(unit
@@
 			(layers "*.Cu" "*.Mask")
 			(remove_unused_layers no)
-			(net "unconnected-(J1-Pin_5-Pad5)")
+			(net "/SCL")
 			(pinfunction "Pin_5_5")
-			(pintype "passive+no_connect")
+			(pintype "passive")
 		)
 		(pad "6" thru_hole circle
@@
 			(layers "*.Cu" "*.Mask")
 			(remove_unused_layers no)
-			(net "unconnected-(J1-Pin_7-Pad7)")
+			(net "/SDA")
 			(pinfunction "Pin_7_7")
-			(pintype "passive+no_connect")
+			(pintype "passive")
 		)
 		(pad "8" thru_hole circle
@@
 			(layers "*.Cu" "*.Mask")
 			(remove_unused_layers no)
-			(net "/SDA")
+			(net "unconnected-(J1-Pin_21-Pad21)")
 			(pinfunction "Pin_21_21")
-			(pintype "passive")
+			(pintype "passive+no_connect")
 		)
 		(pad "22" thru_hole circle
@@
 			(layers "*.Cu" "*.Mask")
 			(remove_unused_layers no)
-			(net "/SCL")
+			(net "unconnected-(J1-Pin_23-Pad23)")
 			(pinfunction "Pin_23_23")
-			(pintype "passive")
+			(pintype "passive+no_connect")
 		)
 		(pad "24" thru_hole circle
@@
 		)
 	)
-	(gr_text "HKU InnoWing IoT Team\n"
+	(gr_text "HKU IoT Beyond Lab\n"
 		(at 106.557 81.427 0)
 		(layer "F.SilkS")
@@
 		)
 	)
-	(gr_text "CrowdAware Node"
+	(gr_text "HKU Thermal Node"
 		(at 106.303 77.871 0)
 		(layer "F.SilkS")
@@
 	(segment
 		(start 101 79.8)
-		(end 101 83.658)
+		(end 101 82.538)
 		(width 0.2)
 		(layer "B.Cu")
@@
 	)
 	(segment
-		(start 101 83.658)
-		(end 100.33 84.328)
+		(start 101 82.538)
+		(end 116.32 82.538)
+		(width 0.2)
+		(layer "B.Cu")
+		(net "/SDA")
+	)
+	(segment
+		(start 116.32 82.538)
+		(end 118.11 84.328)
 		(width 0.2)
 		(layer "B.Cu")
@@
 	(segment
 		(start 96 75.946)
-		(end 96 82.538)
+		(end 96 81.3)
 		(width 0.2)
 		(layer "B.Cu")
@@
 	)
 	(segment
-		(start 96 82.538)
-		(end 97.79 84.328)
+		(start 96 81.3)
+		(end 99.5 81.3)
 		(width 0.2)
 		(layer "B.Cu")
 		(net "/SCL")
 	)
+	(via
+		(at 99.5 81.3)
+		(size 0.8)
+		(drill 0.4)
+		(layers "F.Cu" "B.Cu")
+		(net "/SCL")
+	)
+	(segment
+		(start 99.5 81.3)
+		(end 117.622 81.3)
+		(width 0.2)
+		(layer "F.Cu")
+		(net "/SCL")
+	)
+	(segment
+		(start 117.622 81.3)
+		(end 120.65 84.328)
+		(width 0.2)
+		(layer "F.Cu")
+		(net "/SCL")
+	)

Commit message: Update Rev 1.1 PCB branding
Other:
- board text added: "Designed by Jungheon Kwak based on CrowdAware v1.0"
- board text added: "HKU Innovation Wing IoT Beyond Lab"
- board text added: "Rev 1.1 based on CrowdAware"
- board text added: "Thermal Node Occupancy ML"
- board text removed: "Designed by Ilo Japar"
- board text removed: "HKU IoT Beyond Lab"
- board text removed: "HKU Thermal Node"
- board text removed: "Rev 1.1"
Changed lines of the file:
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@@
 		)
 	)
-	(gr_text "Rev 1.1"
+	(gr_text "Rev 1.1 based on CrowdAware"
 		(at 106.557 79.649 0)
 		(layer "F.SilkS")
@@
 		)
 	)
-	(gr_text "HKU IoT Beyond Lab\n"
+	(gr_text "HKU Innovation Wing IoT Beyond Lab"
 		(at 106.557 81.427 0)
 		(layer "F.SilkS")
@@
 		)
 	)
-	(gr_text "HKU Thermal Node"
+	(gr_text "Thermal Node Occupancy ML"
 		(at 106.303 77.871 0)
 		(layer "F.SilkS")
@@
 		)
 	)
-	(gr_text "Designed by Ilo Japar"
+	(gr_text "Designed by Jungheon Kwak based on CrowdAware v1.0"
 		(at 127.385 64.663 0)
 		(layer "B.SilkS")

Commit message: Add Rev 1.1 hardware test points
Parts:
- added TP1: GND, IoT_Thermal:TestPoint_Plated_Hole_D2.0mm, F.Cu at (78.0, 68.0)
- added TP2: V_EXT, IoT_Thermal:TestPoint_Plated_Hole_D2.0mm, F.Cu at (88.0, 68.0)
- added TP3: SDA, IoT_Thermal:TestPoint_Plated_Hole_D2.0mm, F.Cu at (100.0, 68.0)
- added TP4: SCL, IoT_Thermal:TestPoint_Plated_Hole_D2.0mm, F.Cu at (112.0, 68.0)
Routing:
- net /SDA: track 68.8 -> 78.2 mm
- net /SCL: track 81.5 -> 89.5 mm
- net V_EXT: track 131.8 -> 137.3 mm
Other:
- board text added: "GND"
