File: Hardware/KiCad/HKU Thermal Node Rev1.1.kicad_sch (KiCad schematic)
At the start: 6 parts, among them J1 2 pcs 1x18 socket 2.54mm

Commit message: Fix Rev 1.1 production blockers and rename hardware
Connections:
- net SCL: now also J1.5 (Pin_5); no longer J1.23 (Pin_23)
- net SDA: now also J1.7 (Pin_7); no longer J1.21 (Pin_21)
Other:
- title: CrowdAware Node Rev1.1 -> HKU Thermal Node Rev1.1
Changed lines of the file:
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@@
 	(paper "A5")
 	(title_block
-		(title "CrowdAware Node Rev1.1")
+		(title "HKU Thermal Node Rev1.1")
 		(date "2026-09-16")
 		(rev "1.1")
@@
 	)
 	(no_connect
-		(at 154.94 43.18)
+		(at 154.94 63.5)
 	)
 	(no_connect
@@
 	)
 	(no_connect
-		(at 154.94 45.72)
+		(at 154.94 66.04)
 	)
 	(no_connect
@@
 	(wire
 		(pts
-			(xy 152.4 66.04) (xy 154.94 66.04)
+			(xy 152.4 43.18) (xy 154.94 43.18)
 		)
 		(stroke
@@
 	(wire
 		(pts
-			(xy 152.4 63.5) (xy 154.94 63.5)
+			(xy 152.4 45.72) (xy 154.94 45.72)
 		)
 		(stroke
@@
 	)
 	(label "SDA"
-		(at 152.4 63.5 0)
+		(at 152.4 45.72 0)
 		(effects
 			(font
@@
 	)
 	(label "SCL"
-		(at 152.4 66.04 0)
+		(at 152.4 43.18 0)
 		(effects
 			(font
@@
 		)
 		(instances
-			(project "CrowdAware Node Rev1.1"
+			(project "HKU Thermal Node Rev1.1"
 				(path "/81bee566-7c30-408d-a7cb-e04c7c6916af"
 					(reference "J1")
@@
 		)
 		(instances
-			(project "CrowdAware Node Rev1.1"
+			(project "HKU Thermal Node Rev1.1"
 				(path "/81bee566-7c30-408d-a7cb-e04c7c6916af"
 					(reference "C1")
@@
 		)
 		(instances
-			(project "CrowdAware Node Rev1.1"
+			(project "HKU Thermal Node Rev1.1"
 				(path "/81bee566-7c30-408d-a7cb-e04c7c6916af"
 					(reference "#PWR07")
@@
 		)
 		(instances
-			(project "CrowdAware Node Rev1.1"
+			(project "HKU Thermal Node Rev1.1"
 				(path "/81bee566-7c30-408d-a7cb-e04c7c6916af"
 					(reference "R2")
@@
 		)
 		(instances
-			(project "CrowdAware Node Rev1.1"
+			(project "HKU Thermal Node Rev1.1"
 				(path "/81bee566-7c30-408d-a7cb-e04c7c6916af"
 					(reference "#PWR04")
@@
 		)
 		(instances
-			(project "CrowdAware Node Rev1.1"
+			(project "HKU Thermal Node Rev1.1"
 				(path "/81bee566-7c30-408d-a7cb-e04c7c6916af"
 					(reference "#PWR03")
@@
 		)
 		(instances
-			(project "CrowdAware Node Rev1.1"
+			(project "HKU Thermal Node Rev1.1"
 				(path "/81bee566-7c30-408d-a7cb-e04c7c6916af"
 					(reference "R1")
@@
 		)
 		(instances
-			(project "CrowdAware Node Rev1.1"
+			(project "HKU Thermal Node Rev1.1"
 				(path "/81bee566-7c30-408d-a7cb-e04c7c6916af"
 					(reference "#PWR05")
@@
 		)
 		(instances
-			(project "CrowdAware Node Rev1.1"
+			(project "HKU Thermal Node Rev1.1"
 				(path "/81bee566-7c30-408d-a7cb-e04c7c6916af"
 					(reference "#PWR06")
@@
 		)
 		(instances
-			(project "CrowdAware Node Rev1.1"
+			(project "HKU Thermal Node Rev1.1"
 				(path "/81bee566-7c30-408d-a7cb-e04c7c6916af"
 					(reference "#PWR02")
@@
 		)
 		(instances
-			(project "CrowdAware Node Rev1.1"
+			(project "HKU Thermal Node Rev1.1"
 				(path "/81bee566-7c30-408d-a7cb-e04c7c6916af"
 					(reference "#PWR01")
@@
 		)
 		(instances
-			(project "CrowdAware Node Rev1.1"
+			(project "HKU Thermal Node Rev1.1"
 				(path "/81bee566-7c30-408d-a7cb-e04c7c6916af"
 					(reference "A1")
@@
 		)
 		(instances
-			(project "CrowdAware Node Rev1.1"
+			(project "HKU Thermal Node Rev1.1"
 				(path "/81bee566-7c30-408d-a7cb-e04c7c6916af"
 					(reference "C2")

Commit message: Add Rev 1.1 hardware test points
Parts:
- added TP1: GND, IoT_Thermal:TestPoint_Plated_Hole_D2.0mm, symbol IoT_Thermal:TestPoint
- added TP2: V_EXT, IoT_Thermal:TestPoint_Plated_Hole_D2.0mm, symbol IoT_Thermal:TestPoint
- added TP3: SDA, IoT_Thermal:TestPoint_Plated_Hole_D2.0mm, symbol IoT_Thermal:TestPoint
- added TP4: SCL, IoT_Thermal:TestPoint_Plated_Hole_D2.0mm, symbol IoT_Thermal:TestPoint
Connections:
- net GND: now also TP1.1
- net SCL: now also TP4.1
- net SDA: now also TP3.1
- net V_EXT: now also TP2.1
